File: Nano shield for arduino-thermal.kicad_pcb (KiCad board)
At the start: 2 copper layers, 12 parts, among them J1 Conn_01x03_Male, J2 Conn_01x03_Male, J3 Conn_01x16_Female, J4 Barrel_Jack, J5 Conn_01x21_Male

Commit message: Revision 2.0
Other:
- board text added: "Arduino-Thermal board rev 2.0"
- board text removed: "Arduino-Thermal board rev2"
Changed lines of the file:
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@@
     (effects (font (size 1 1) (thickness 0.15)))
   )
-  (gr_text "Arduino-Thermal\nboard rev2" (at 129.21 61.09) (layer "F.SilkS")
+  (gr_text "Arduino-Thermal\nboard rev 2.0" (at 129.21 61.09) (layer "F.SilkS")
     (effects (font (size 1.5 1.75) (thickness 0.375) italic))
   )

Commit message: Revision 2.1.1 - Some paths have been changed
Parts:
- J5: value Conn_01x21_Male -> Conn_01x25_Male; footprint Connector_PinHeader_2.54mm:PinHeader_1x21_P2.54mm_Vertical -> Connector_PinHeader_2.54mm:PinHeader_1x25_P2.54mm_Vertical
Connections:
- A1 pad 18: Net-(A1-Pad18) -> unconnected-(A1-Pad18)
- A1 pad 28: Net-(A1-Pad28) -> unconnected-(A1-Pad28)
- A1 pad 3: Net-(A1-Pad3) -> unconnected-(A1-Pad3)
- J3 pad 10: Net-(J3-Pad10) -> unconnected-(J3-Pad10)
- J3 pad 7: Net-(J3-Pad7) -> unconnected-(J3-Pad7)
- J3 pad 8: Net-(J3-Pad8) -> unconnected-(J3-Pad8)
- J3 pad 9: Net-(J3-Pad9) -> unconnected-(J3-Pad9)
- J5 pad 18: Net-(J3-Pad15) -> GND
- J5 pad 19: +5V -> Net-(J3-Pad15)
- J5 pad 20: Net-(A1-Pad30) -> Net-(J3-Pad15)
- J5 pad 21: Net-(J4-Pad1) -> +5V
Routing:
- net Net-(J1-Pad2): track 46.9 -> 59.7 mm
- net Net-(J4-Pad1): track 85.3 -> 75.8 mm, vias 0 -> 2
- net Net-(A1-Pad30): track 18.2 -> 11.4 mm
- net Net-(J3-Pad3): track 51.9 -> 54.9 mm
- net Net-(A1-Pad19): track 38.6 -> 41.1 mm
- net +5V: track 145.7 -> 143.5 mm
- net Net-(J3-Pad15): track 91.5 -> 90.2 mm
- net Net-(A1-Pad20): track 38.6 -> 39.9 mm
- net Net-(A1-Pad24): track 38.6 -> 39.9 mm
- net Net-(A1-Pad23): track 38.6 -> 39.9 mm
- net Net-(A1-Pad21): track 38.6 -> 39.9 mm
- net Net-(A1-Pad22): track 38.6 -> 39.9 mm
- net Net-(A1-Pad2): track 51.9 -> 52.8 mm
- net Net-(A1-Pad1): track 47.9 -> 48.8 mm
- net Net-(A1-Pad25): track 38.6 -> 39.5 mm
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Other:
- board text added: "Arduino-Thermal board rev 2.1.1"
- board text added: "LED"
- board text added: "SW"
- board text removed: "Arduino-Thermal board rev 2.0"
